File: hardware/kicad/MOD-0011.kicad_pcb (KiCad board)
At the start: 2 copper layers, 80 x 40 mm, 127 parts, among them J1 USB-C USB (Power), J10 Cluster B, J11 Cluster C, J12 Cluster D, J13 Cluster C, J14 noknok_Pico_Socket_P1-20, J15 noknok_Pico_Socket_P21-40, J2 USB-C USB (host), J3 JST SH port 1 (bus A), J4 JST SH port 2 (bus A), J5 JST SH port 3 (bus B), J6 JST SH port 4 (bus B), J8 SWD pads, J9 Cluster A, U1 CH32X035G8U6, U11 noknok_SY6280AAC, U2 TPS54302, U3 noknok_SY6280AAC, U4 INA180A2, U5 noknok_ME6203A33M3G, U6 noknok_AP2114H-3.3, U7 noknok_SY6280AAC, U8 noknok_SY6280AAC, U9 noknok_AP2114H-3.3

Commit message: DEV-45: rev 1.1 - R39/R40 5.1k pull-downs on USB_DP/USB_DN at the Pico (RP2350 erratum E9), schematic note, layout (D16/D17 shifted 1.75 mm), BOM line 20 now R1,R2,R39,R40 x4 (C23186)
ERC 0. DRC: the 12 known board-edge items only, 0 unconnected, schematic parity 0.
BOM cross-checked against the schematic: 115 parts each.
Parts:
- added R39: 5.1k, Resistor_SMD:R_0603_1608Metric, F.Cu at (162.8, 93.8)
- added R40: 5.1k, Resistor_SMD:R_0603_1608Metric, F.Cu at (159.7, 93.5)
- moved D16 1.75 mm to (134.8, 114.8)
- moved D17 1.75 mm to (134.8, 116.3)
Routing:
- net GND: track 257.4 -> 274.3 mm
- net USB_DN: track 15.5 -> 24.4 mm
- net USB_DP: track 15.4 -> 24.3 mm
- net +5V: track 119.1 -> 117.2 mm
Other:
- board text added: "B"
- board text added: "I2C"
- board text added: "MCU Flash"
- board text added: "PWR in"
- board text added: "Pico USB-Port here"
- board text added: "Pico WLAN here"
- board text added: "Pls read the manual at https://noknok.app"
- board text removed: "I2C-B"
- board text removed: "Pico orientation: USB Port this side"
- board text removed: "Pico orientation: WLAN antenna this side"

Commit message: MOD-0011 rev 1.1 labels: silkscreen "Rev 1.1 / Oct 26", schematic title block rev 1.1 (2026-10-23), schematic PDF re-exported
ERC 0. DRC: the 12 known board-edge items only, 0 unconnected, schematic parity 0. No parts or tracks changed.
Other:
- board text added: "MOD-0011 Rev 1.1 Oct 26"
- board text removed: "MOD-0011 Rev 1.0 Sep 26"
Changed lines of the file:
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@@
 		(layer "Edge.Cuts")
 	)
-	(gr_text "MOD-0011\nRev 1.0\nSep 26"
+	(gr_text "MOD-0011\nRev 1.1\nOct 26"
 		(at 147.6 84.3 0)
 		(layer "F.SilkS")
